File: eagle/NJM2936+MAU106_PSU/NJM2936+MAU106_PSU.brd (EAGLE design)
At the start: 93.7 x 71.1 mm, 28 parts, among them CN1 PWIN, CN2 DPWR, CN3 DPWR, CN4 DPWR, CN5 DPWR, IC1 NJM2396V, IC2 MAU106

Commit message: Add some image files
Routing:
- net N$2: track 60.3 -> 55.2 mm
- net D+5V: track 119.1 -> 123.3 mm
Changed lines of the file:
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@@
 <wire x1="50.8" y1="7.62" x2="50.8" y2="7.7" width="0.4064" layer="16"/>
 <wire x1="50.8" y1="7.7" x2="48.3" y2="10.2" width="0.4064" layer="16"/>
-<wire x1="48.26" y1="53.34" x2="48.26" y2="50.8" width="0.4064" layer="16"/>
-<wire x1="48.26" y1="50.8" x2="48.26" y2="25.44" width="0.4064" layer="16"/>
 <wire x1="48.26" y1="25.44" x2="48.3" y2="25.4" width="0.4064" layer="16"/>
-<wire x1="60.96" y1="53.34" x2="58.42" y2="50.8" width="0.4064" layer="16"/>
-<wire x1="58.42" y1="50.8" x2="48.26" y2="50.8" width="0.4064" layer="16"/>
 <wire x1="17.78" y1="15.24" x2="20.32" y2="15.24" width="0.4064" layer="16"/>
+<wire x1="48.26" y1="25.44" x2="48.26" y2="40.64" width="0.4064" layer="16"/>
+<wire x1="48.26" y1="40.64" x2="60.96" y2="53.34" width="0.4064" layer="16"/>
+<wire x1="48.26" y1="53.34" x2="48.26" y2="40.64" width="0.4064" layer="16"/>
 </signal>
 <signal name="A-5V">
@@
 <wire x1="27.94" y1="20.32" x2="27.94" y2="15.24" width="0.4064" layer="16"/>
 <wire x1="22.86" y1="30.48" x2="35.56" y2="30.48" width="0.4064" layer="16"/>
-<wire x1="35.56" y1="30.48" x2="35.56" y2="17.78" width="0.4064" layer="16"/>
-<wire x1="35.56" y1="17.78" x2="33.02" y2="15.24" width="0.4064" layer="16"/>
-<wire x1="33.02" y1="15.24" x2="27.94" y2="15.24" width="0.4064" layer="16"/>
 <wire x1="35.48" y1="45.49" x2="35.48" y2="30.56" width="0.4064" layer="16"/>
 <wire x1="35.48" y1="30.56" x2="35.56" y2="30.48" width="0.4064" layer="16"/>
+<wire x1="35.56" y1="30.48" x2="35.56" y2="22.86" width="0.4064" layer="16"/>
+<wire x1="35.56" y1="22.86" x2="33.02" y2="20.32" width="0.4064" layer="16"/>
+<wire x1="33.02" y1="20.32" x2="27.94" y2="20.32" width="0.4064" layer="16"/>
 </signal>
 <signal name="N$3">
